File: KiCad shield files/penshield.sch (KiCad schematic (older format))
At the start: 7 parts, among them P1 To Battery, P2 Servo A, P3 Arduino PWM pins, P4 Servo B, P5 Servo C, P6 Arduino Power Pins, SW1 Switch_SPDT_x2

Commit message: Updated KiCad project; fixed spacing of header pins on shield
Parts:
- SW1: symbol Switch_SPDT_x2 -> Switch_SPDT_x2-RESCUE-penshield
Changed lines of the file:
@@
 EESchema Schematic File Version 2
+LIBS:penshield-rescue
 LIBS:power
 LIBS:device
@@
 Connection ~ 3300 1850
 $Comp
-L Switch_SPDT_x2 SW1
+L Switch_SPDT_x2-RESCUE-penshield SW1
 U 2 1 571DBD8A
 P 3000 2900
@@
 $EndComp
 $Comp
-L Switch_SPDT_x2 SW1
+L Switch_SPDT_x2-RESCUE-penshield SW1
 U 1 1 571DBDC5
 P 2100 1950
